File: raven-caller/_autosave-raven-caller.kicad_pcb (KiCad board)
At the start: 2 copper layers, 80.6 x 31.1 mm, 51 parts, among them J1 I2C LCD, J2 Conn_01x02_Pin, J3 Conn_Coaxial, J7 USB_C_Receptacle_USB2.0_16P, Q1 BSS138, SW1 RotaryEncoder_Switch, SW2 SW_SPDT, U10 TPD1E05U06DYA, U11 TXS0102DCT, U12 XIAO-SAMD21-DIP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

Commit message: final pcb(i hope)
Routing:
- net GND: vias 180 -> 117
