File: raven-caller/raven-caller.kicad_pcb (KiCad board)
At the start: 2 copper layers, 80.6 x 31.1 mm, 51 parts, among them J1 I2C LCD, J2 Conn_01x02_Pin, J3 Conn_Coaxial, J7 USB_C_Receptacle_USB2.0_16P, Q1 BSS138, SW1 RotaryEncoder_Switch, SW2 SW_SPDT, U10 TPD1E05U06DYA, U11 TXS0102DCT, U12 XIAO-SAMD21-DIP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

Commit message: final fixes
Parts:
- added G***: LOGO, EAOLogo:eaologoSMALL, F.Cu at (167.0, 116.4)
- moved H1 0.30 mm to (196.3, 119.5)
- moved H2 0.30 mm to (196.3, 94.1)
Routing:
- net GND: track 114.5 -> 120.3 mm, vias 180 -> 136
Other:
- board text added: "EAO 2025 Raven Caller V1"
